File: rf_chain.kicad_sch (KiCad schematic)
At the start: 36 parts, among them U2 PE43712B-Z, U3 TRF37D73, U4 XLF-172H+, U6 TRF37D73, U8 RCAT-01+

Commit message: Change SMA to edge-launch
Parts:
- SH1: footprint My_Footprints:MS593-10F -> My_Footprints:MS593-10F_Two_Mouseholes_2x1mm
Changed lines of the file:
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@@
 			)
 		)
-		(property "Footprint" "My_Footprints:MS593-10F"
+		(property "Footprint" "My_Footprints:MS593-10F_Two_Mouseholes_2x1mm"
 			(at 369.57 194.31 0)
 			(effects

Commit message: Finish preliminary routing of one channel
Parts:
- added U5: RCAT-01+, My_Footprints:RCAT_LZ1737, symbol My_Symbols:RCAT-01+
Connections:
- net GND: now also SH1.1 (Shield), U5.2 (GND), U5.4 (GND)
- net at C20.1: now also U5.3 (RF_OUT); no longer U4.16 (RF-OUT)
- new net: U4.16 (RF-OUT), U5.1 (RF_IN)
Other:
- moved on the sheet: C1, C10, C11, C15, C19, C2, C20, C21, C22, C23, C24, C3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

Commit message: Add part numbers for BOM
Parts:
- C1, C23: value 1uF -> 1u; MFG (none) -> TDK; MFG_PN (none) -> C1608X7R1E105K080AE; Price (none) -> 0.1
- C10: MFG (none) -> Murata; MFG_PN (none) -> GRM1885C1H103JA01D; Price (none) -> 0.04
- C11, C15, C19, C5: MFG (none) -> Kyocera AVX; MFG_PN (none) -> 600S130FT250XTV; Price (none) -> 1.57
- C2, C22: MFG (none) -> Murata; MFG_PN (none) -> GRM1885C1H103JA01D; Price (none) -> .04
- C20, C24, C4, C6, C7: MFG (none) -> Murata; MFG_PN (none) -> GCM1555C1H102FA16D; Price (none) -> 0.03
- C21, C3: MFG (none) -> Kyocera; MFG_PN (none) -> KGM15ACG1H101FT; Price (none) -> .04
- C9: MFG (none) -> Murata; MFG_PN (none) -> GCJ188R71E104KA12D; Price (none) -> 0.01
- R1: MFG (none) -> Panasonic; MFG_PN (none) -> ERJ-3EKF1002V; Price (none) -> 0.01
- R10, R11, R12, R13, R3, R4, R8, R9: MFG (none) -> Vishay Dale Thin Film; MFG_PN (none) -> FCHP0402E50R0BGT1; Price (none) -> 1.58
- U2: MFG (none) -> pSemi; MFG_PN (none) -> PE43712B-Z; Price (none) -> 7.05
- U3, U6: MFG (none) -> TI; MFG_PN (none) -> TRF37D73IDSGR; Price (none) -> 1.24
- U4: MFG (none) -> Mini-Circuits; MFG_PN (none) -> XLF-172H+; Price (none) -> 19.64
- U5, U8: MFG MiniCircuits -> Mini-Circuits; Price (none) -> 19.25

Commit message: Update RF shield
Parts:
- removed SH1: RFShield_TwoPieces, My_Footprints:MS593-10F_Two_Mouseholes_2x1mm, symbol Device:RFShield_TwoPieces
